Commit message: adding camera

File: model/urdf/robot.xacro (robot description, xacro)
@@ -244,33 +244,31 @@
     </sensor>
   </gazebo> -->
-  <!--CAMERA CRAFT-->
-  <!-- <link name="Camera">
-    <visual>
-      <origin rpy="0 0 0" xyz="0 0 0"/>
-      <geometry>
-        <mesh filename="package://robot_diff_description/meshes/Camera.stl"/>
-      </geometry>
-    </visual>
-    <collision>
-      <origin rpy="0 0 0" xyz="0 0 0"/>
-      <geometry>
-        <mesh filename="package://robot_diff_description/meshes/Camera.stl"/>
-      </geometry>
-    </collision>
-    <inertial>
-      <origin rpy="0 0 0" xyz="0 0 0"/>
-      <mass value="0.002"/>
+  <link name="camera">
+    <visual>
+      <origin rpy="0 0 0" xyz="0 0 0"/>
+      <geometry>
+        <mesh filename="file:///home/tecchio/code/catkin_learnbotics/src/learnrobotics/model/stl/Camera.stl"/>
+      </geometry>
+    </visual>
+    <collision>
+      <origin rpy="0 0 0" xyz="0 0 0"/>
+      <geometry>
+        <mesh filename="file:///home/tecchio/code/catkin_learnbotics/src/learnrobotics/model/stl/Camera.stl"/>
+      </geometry>
+    </collision>
+    <inertial>
+      <origin rpy="0 0 0" xyz="0 0 0"/>
+      <mass value="0.02"/>
       <inertia ixx="1.397e-7" ixy="0" ixz="-2.070e-12" iyy="1.512e-7" iyz="1.844e-9" izz="7.943e-8"/>
     </inertial>
   </link>
-  <joint name="Lidar_to_Camera" type="fixed">
-    <parent link="Lidar"/>
-    <child link="Camera"/>
-    <origin rpy="0 0 -1.571" xyz="0 -0.00591798 0.03857247"/>
-  </joint> -->
-  <!--CAMERA SENSOR-->
-  <!-- <gazebo reference="Camera">
+  <joint name="chassis_to_camera" type="fixed">
+    <parent link="chassis"/>
+    <child link="camera"/>
+    <origin rpy="0 0 0" xyz="0.07456502 0 0.03016464"/>
+  </joint>
+  <gazebo reference="camera">
     <sensor type="camera" name="camera_top">
-      <update_rate>30.0</update_rate>
+      <update_rate>60.0</update_rate>
       <camera name="head">
         <horizontal_fov>1.3962634</horizontal_fov>
@@ -288,8 +286,8 @@
         <alwaysOn>true</alwaysOn>
         <updateRate>0.0</updateRate>
-        <cameraName>diff/camera_top</cameraName>
+        <cameraName>camera_top</cameraName>
         <imageTopicName>image_raw</imageTopicName>
         <cameraInfoTopicName>camera_info</cameraInfoTopicName>
-        <frameName>Camera</frameName>
+        <frameName>camera</frameName>
         <hackchassisline>0.07</hackchassisline>
         <distortionK1>0.0</distortionK1>
@@ -300,5 +298,5 @@
       </plugin>
     </sensor>
-  </gazebo> -->
+  </gazebo>
   <gazebo>
     <plugin name="gazebo_ros_control" filename="libgazebo_ros_diff_drive.so">

Commit message: using dataspeed inc velodyne plugin

File: model/urdf/robot.xacro (robot description, xacro)
@@ -187,61 +187,10 @@
     <material>Gazebo/Green</material>
   </gazebo>
-  <!--LIDAR CRAFT-->
-  <!-- <link name="Lidar">
-    <visual>
-      <origin rpy="0 0 0" xyz="0 0 0"/>
-      <geometry>
-        <mesh filename="package://robot_diff_description/meshes/Lidar.stl"/>
-      </geometry>
-    </visual>
-    <collision>
-      <origin rpy="0 0 0" xyz="0 0 0"/>
-      <geometry>
-        <mesh filename="package://robot_diff_description/meshes/Lidar.stl"/>
-      </geometry>
-    </collision>
-    <inertial>
-      <origin rpy="0 0 0" xyz="0 0 0"/>
-      <mass value="0.031"/>
-      <inertia ixx="1.184e-5" ixy="-4.274e-11" ixz="-2.070e-12" iyy="1.206e-5" iyz="0" izz="4.594e-6"/>
-    </inertial>
-  </link>
-  <joint name="chassis_to_Lidar" type="fixed">
-    <parent link="chassis"/>
-    <child link="Lidar"/>
-    <origin rpy="-1.571 1.571 0" xyz="0 0.07911977 0"/>
-  </joint> -->
-  <!-- RAY SENSOR CRAFT -->
-  <!-- <gazebo reference="Lidar">
-    <sensor type="ray" name="head_hokuyo_sensor">
-      <pose>0 0 0 0 0 0</pose>
-      <visualize>false</visualize>
-      <update_rate>20</update_rate>
-      <ray>
-        <scan>
-          <horizontal>
-            <samples>720</samples>
-            <resolution>1</resolution>
-            <min_angle>3.1415</min_angle>
-            <max_angle>6.2831</max_angle>
-          </horizontal>
-        </scan>
-        <range>
-          <min>0.10</min>
-          <max>10.0</max>
-          <resolution>0.01</resolution>
-        </range>
-        <noise>
-          <type>gaussian</type>
-          <mean>0.0</mean>
-          <stddev>0.01</stddev>
-        </noise>
-      </ray>
-      <plugin name="gazebo_ros_head_hokuyo_controller" filename="libgazebo_ros_laser.so">
-        <topicName>/diff/laser/scan</topicName>
-        <frameName>Lidar</frameName>
-      </plugin>
-    </sensor>
-  </gazebo> -->
+  <xacro:arg name="gpu" default="true"/>
+  <xacro:property name="gpu" value="$(arg gpu)" />
+  <xacro:include filename="$(find velodyne_description)/urdf/VLP-16.urdf.xacro"/>
+  <VLP-16 parent="chassis" name="velodyne" topic="/velodyne_points" hz="10" samples="440" gpu="${gpu}">
+    <origin xyz="0 0 0.045" rpy="0 0 0" />
+  </VLP-16>
   <link name="camera">
     <visual>
